File: hw/lipo_status.brd (EAGLE design)
At the start: 39 x 23.2 mm, 36 parts, among them IC1 LM317-3V3

Commit message: removed tracking of eagle backup files\nadapted SW\nadapted schematic and layout
Parts:
- R19: value 10k -> 100k
- R20: value 1k3 -> 13k
Changed lines of the file:
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@@
 <attribute name="TP_SIGNAL_NAME" value="" x="32.5" y="6.1" size="1.778" layer="27" display="off"/>
 </element>
-<element name="R19" library="rcl" package="R0603" value="10k" x="21.4" y="17.8" rot="MR180"/>
-<element name="R20" library="rcl" package="R0603" value="1k3" x="23.1" y="19.4" rot="MR180"/>
+<element name="R19" library="rcl" package="R0603" value="100k" x="21.4" y="17.8" rot="MR180"/>
+<element name="R20" library="rcl" package="R0603" value="13k" x="23.1" y="19.4" rot="MR180"/>
 </elements>
 <signals>

Commit message: added gerber files
Parts:
- added R21: 10k, rcl:R0603
- added T1: IRLML5203TRPBF, SchlegelAr_Master:SOT23
- moved IC1 1.60 mm to (9.70, 17.3)
- moved LED1 1.60 mm to (32.0, 20.3)
- moved LED2 1.60 mm to (32.0, 18.6)
- moved R1 1.60 mm to (28.6, 20.3)
- moved R12 1.60 mm to (15.0, 19.1)
- moved R13 1.60 mm to (28.5, 20.3)
- moved R14 1.60 mm to (28.5, 18.6)
- moved R18 1.60 mm to (19.2, 17.1)
- moved R2 1.60 mm to (28.6, 18.6)
- moved R20 1.60 mm to (23.1, 21.0)
- moved TP2 1.60 mm to (32.5, 7.70)
- moved C1 1.60 mm to (16.5, 16.2)
- moved JP1 1.60 mm to (36.3, 11.6)
- moved JP2 1.60 mm to (2.40, 11.6)
- moved LED4 1.60 mm to (32.0, 15.2)
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Connections:
- new net N$19: R21.1, T1.1
- new net N$20: C2.1, IC1.3, T1.2
- net GND: now also R21.2
- net VCC: now also T1.3; no longer C2.1, IC1.3
Routing:
- net N$20: track 0.00 -> 7.84 mm, vias 0 -> 1
- net VCC: track 43.5 -> 37.1 mm, vias 1 -> 0
- net N$19: track 0.00 -> 1.67 mm
Other:
- board text added: "Armin Schlegel"
- board text added: "LIPO_STATUS, V1"
- board text added: "Out"
- board text added: "bot"
- board text added: "top"
- board text removed: "out"
